File: DronePCB/mic.kicad_sch (KiCad schematic)
At the start: 4 parts

Commit message: Completed H-Bridge Circuit | Finished Schematic | Working on pcb design
Parts:
- C16: renamed from C17; footprint (none) -> Capacitor_SMD:C_0603_1608Metric
- C17: renamed from C16; footprint (none) -> Capacitor_SMD:C_0603_1608Metric
- MK1: footprint DMM-4026-B-I2S-R:MIC_DMM-4026-B-I2S-R -> ExternalParts:MIC_DMM-4026-B-I2S-R
- R4: renamed from R2; footprint (none) -> Resistor_SMD:R_0603_1608Metric
Changed lines of the file:
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@@
 		(in_pos_files yes)
 		(dnp no)
-		(property "Reference" "C16"
+		(property "Reference" "C17"
 			(at 167.64 96.012 90)
 			(show_name no)
@@
 			)
 		)
-		(property "Footprint" ""
+		(property "Footprint" "Capacitor_SMD:C_0603_1608Metric"
 			(at 171.45 91.1352 0)
 			(hide yes)
@@
 			(project "DronePCB"
 				(path "/c9b74494-ac48-4f27-9459-39f0e04d9d05/93a7ea6a-fcf4-476b-8d2c-922c1c402e60"
-					(reference "C16")
+					(reference "C17")
 					(unit 1)
 				)
@@
 			)
 		)
-		(property "Footprint" "DMM-4026-B-I2S-R:MIC_DMM-4026-B-I2S-R"
+		(property "Footprint" "ExternalParts:MIC_DMM-4026-B-I2S-R"
 			(at 138.43 97.79 0)
 			(hide yes)
@@
 		(dnp no)
 		(fields_autoplaced yes)
-		(property "Reference" "#PWR011"
+		(property "Reference" "#PWR022"
 			(at 119.38 107.95 0)
 			(hide yes)
@@
 			(project "DronePCB"
 				(path "/c9b74494-ac48-4f27-9459-39f0e04d9d05/93a7ea6a-fcf4-476b-8d2c-922c1c402e60"
-					(reference "#PWR011")
+					(reference "#PWR022")
 					(unit 1)
 				)
@@
 		(dnp no)
 		(fields_autoplaced yes)
-		(property "Reference" "#PWR010"
+		(property "Reference" "#PWR025"
 			(at 173.99 114.3 0)
 			(hide yes)
@@
 			(project "DronePCB"
 				(path "/c9b74494-ac48-4f27-9459-39f0e04d9d05/93a7ea6a-fcf4-476b-8d2c-922c1c402e60"
-					(reference "#PWR010")
+					(reference "#PWR025")
 					(unit 1)
 				)
@@
 		(dnp no)
 		(fields_autoplaced yes)
-		(property "Reference" "#PWR09"
+		(property "Reference" "#PWR023"
 			(at 157.48 113.03 0)
 			(hide yes)
@@
 			(project "DronePCB"
 				(path "/c9b74494-ac48-4f27-9459-39f0e04d9d05/93a7ea6a-fcf4-476b-8d2c-922c1c402e60"
-					(reference "#PWR09")
+					(reference "#PWR023")
 					(unit 1)
 				)
@@
 		(dnp no)
 		(fields_autoplaced yes)
-		(property "Reference" "#PWR012"
+		(property "Reference" "#PWR024"
 			(at 173.99 96.52 0)
 			(hide yes)
@@
 			(project "DronePCB"
 				(path "/c9b74494-ac48-4f27-9459-39f0e04d9d05/93a7ea6a-fcf4-476b-8d2c-922c1c402e60"
-					(reference "#PWR012")
+					(reference "#PWR024")
 					(unit 1)
 				)
@@
 		(dnp no)
 		(fields_autoplaced yes)
-		(property "Reference" "R2"
+		(property "Reference" "R4"
 			(at 176.53 101.5999 0)
 			(show_name no)
@@
 			)
 		)
-		(property "Footprint" ""
+		(property "Footprint" "Resistor_SMD:R_0603_1608Metric"
 			(at 175.006 103.124 90)
 			(hide yes)
@@
 			(project "DronePCB"
 				(path "/c9b74494-ac48-4f27-9459-39f0e04d9d05/93a7ea6a-fcf4-476b-8d2c-922c1c402e60"
-					(reference "R2")
+					(reference "R4")
 					(unit 1)
 				)
@@
 		(dnp yes)
 		(fields_autoplaced yes)
-		(property "Reference" "C17"
+		(property "Reference" "C16"
 			(at 167.64 76.2 90)
 			(show_name no)
@@
 			)
 		)
-		(property "Footprint" ""
+		(property "Footprint" "Capacitor_SMD:C_0603_1608Metric"
 			(at 171.45 82.8548 0)
 			(hide yes)
@@
 			(project "DronePCB"
 				(path "/c9b74494-ac48-4f27-9459-39f0e04d9d05/93a7ea6a-fcf4-476b-8d2c-922c1c402e60"
-					(reference "C17")
+					(reference "C16")
 					(unit 1)
 				)
