File: DronePCB/HBridge.kicad_sch (KiCad schematic)
At the start: 30 parts, among them M1 Motor_DC, M2 Motor_DC, Q10 AO3401A, Q11 AO3401A, Q8 AO3401A, Q9 AO3401A, U10 DRV8231DDAR, U9 DRV8231DDAR

Commit message: finished H bridge pcb design
Parts:
- removed R48: 100, Resistor_SMD:R_0603_1608Metric, symbol Device:R_US
- removed R49: 10k, Resistor_SMD:R_0603_1608Metric, symbol Device:R_US
Changed lines of the file:
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@@
-	)
-	(symbol
-		(lib_id "Device:R_US")
-		(at 101.6 223.52 90)
-		(mirror x)
-		(unit 1)
-		(body_style 1)
-		(exclude_from_sim no)
-		(in_bom yes)
-		(on_board yes)
-		(in_pos_files yes)
-		(dnp no)
-		(property "Reference" "R48"
-			(at 101.6 228.6 90)
-			(show_name no)
-			(do_not_autoplace no)
-			(effects
-				(font
-					(size 1.27 1.27)
-				)
-			)
-		)
-		(property "Value" "100"
-			(at 101.6 226.06 90)
-			(show_name no)
-			(do_not_autoplace no)
-			(effects
-				(font
-					(size 1.27 1.27)
-				)
-			)
-		)
-		(property "Footprint" "Resistor_SMD:R_0603_1608Metric"
-			(at 101.854 224.536 90)
-			(hide yes)
-			(show_name no)
-			(do_not_autoplace no)
-			(effects
-				(font
-					(size 1.27 1.27)
-				)
-			)
-		)
-		(property "Datasheet" ""
-			(at 101.6 223.52 0)
-			(hide yes)
-			(show_name no)
-			(do_not_autoplace no)
-			(effects
-				(font
-					(size 1.27 1.27)
-				)
-			)
-		)
-		(property "Description" "Resistor, US symbol"
-			(at 101.6 223.52 0)
-			(hide yes)
-			(show_name no)
-			(do_not_autoplace no)
-			(effects
-				(font
-					(size 1.27 1.27)
-				)
-			)
-		)
-		(pin "2"
-		)
-		(pin "1"
-		)
-		(instances
-			(project "DronePCB"
-				(path "/c9b74494-ac48-4f27-9459-39f0e04d9d05/064430ba-d2ef-4218-b13a-03feb27628bb"
-					(reference "R48")
-					(unit 1)
-				)
-			)
-		)
 	)
 	(symbol
@@
 					(unit 1)
 				)
-			)
-		)
-	)
-	(symbol
-		(lib_id "Device:R_US")
-		(at 106.68 231.14 0)
-		(mirror x)
-		(unit 1)
-		(body_style 1)
-		(exclude_from_sim no)
-		(in_bom yes)
-		(on_board yes)
-		(in_pos_files yes)
-		(dnp no)
-		(property "Reference" "R49"
-			(at 109.22 232.41 0)
-			(show_name no)
-			(do_not_autoplace no)
-			(effects
-				(font
-					(size 1.27 1.27)
-				)
-				(justify left)
-			)
-		)
-		(property "Value" "10k"
-			(at 109.22 229.8701 0)
-			(show_name no)
-			(do_not_autoplace no)
-			(effects
-				(font
-					(size 1.27 1.27)
-				)
-				(justify left)
-			)
-		)
-		(property "Footprint" "Resistor_SMD:R_0603_1608Metric"
-			(at 107.696 230.886 90)
-			(hide yes)
-			(show_name no)
-			(do_not_autoplace no)
-			(effects
-				(font
-					(size 1.27 1.27)
-				)
-			)
-		)
-		(property "Datasheet" ""
-			(at 106.68 231.14 0)
-			(hide yes)
-			(show_name no)
-			(do_not_autoplace no)
-			(effects
-				(font
-					(size 1.27 1.27)
-				)
-			)
-		)
-		(property "Description" "Resistor, US symbol"
-			(at 106.68 231.14 0)
-			(hide yes)
-			(show_name no)
-			(do_not_autoplace no)
-			(effects
-				(font
-					(size 1.27 1.27)
-				)
-			)
-		)
-		(pin "2"
-		)
-		(pin "1"
-		)
-		(instances
-			(project "DronePCB"
-				(path "/c9b74494-ac48-4f27-9459-39f0e04d9d05/064430ba-d2ef-4218-b13a-03feb27628bb"
-					(reference "R49")
-					(unit 1)
-				)

Commit message: All circuits complete
Parts:
- renumbered C46 to C50, C47 to C51, C48 to C52, C49 to C53, C50 to C54, C51 to C55, C52 to C56, C53 to C57, Q8 to Q6, Q9 to Q7, Q10 to Q8, Q11 to Q9, R45 to R36, R42 to R37, R44 to R38, R50 to R39, R46 to R40, R35 to R42, R36 to R43, R37 to R44, R38 to R45, R39 to R46, R40 to R47
Changed lines of the file:
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@@
 		(dnp no)
 		(fields_autoplaced yes)
-		(property "Reference" "R35"
+		(property "Reference" "R42"
 			(at 109.22 49.53 90)
 			(show_name no)
@@
 			(project "DronePCB"
 				(path "/c9b74494-ac48-4f27-9459-39f0e04d9d05/064430ba-d2ef-4218-b13a-03feb27628bb"
-					(reference "R35")
+					(reference "R42")
 					(unit 1)
 				)
@@
 		(dnp no)
 		(fields_autoplaced yes)
-		(property "Reference" "R37"
+		(property "Reference" "R44"
 			(at 109.22 127 90)
 			(show_name no)
@@
 			(project "DronePCB"
 				(path "/c9b74494-ac48-4f27-9459-39f0e04d9d05/064430ba-d2ef-4218-b13a-03feb27628bb"
-					(reference "R37")
+					(reference "R44")
 					(unit 1)
 				)
@@
 		(in_pos_files yes)
 		(dnp no)
-		(property "Reference" "Q8"
+		(property "Reference" "Q6"
 			(at 119.38 44.4499 0)
 			(show_name no)
@@
 			(project "DronePCB"
 				(path "/c9b74494-ac48-4f27-9459-39f0e04d9d05/064430ba-d2ef-4218-b13a-03feb27628bb"
-					(reference "Q8")
+					(reference "Q6")
 					(unit 1)
 				)
@@
 		(dnp no)
 		(fields_autoplaced yes)
-		(property "Reference" "#PWR067"
+		(property "Reference" "#PWR069"
 			(at 181.61 162.56 0)
 			(hide yes)
@@
 			(project "DronePCB"
 				(path "/c9b74494-ac48-4f27-9459-39f0e04d9d05/064430ba-d2ef-4218-b13a-03feb27628bb"
-					(reference "#PWR067")
+					(reference "#PWR069")
 					(unit 1)
 				)
@@
 		(in_pos_files yes)
 		(dnp yes)
-		(property "Reference" "C46"
+		(property "Reference" "C50"
 			(at 127 39.7509 0)
 			(show_name no)
@@
 			(project "DronePCB"
 				(path "/c9b74494-ac48-4f27-9459-39f0e04d9d05/064430ba-d2ef-4218-b13a-03feb27628bb"
-					(reference "C46")
+					(reference "C50")
 					(unit 1)
 				)
@@
 		(in_pos_files yes)
 		(dnp no)
-		(property "Reference" "R36"
+		(property "Reference" "R43"
 			(at 109.22 64.77 90)
 			(show_name no)
@@
 			(project "DronePCB"
 				(path "/c9b74494-ac48-4f27-9459-39f0e04d9d05/064430ba-d2ef-4218-b13a-03feb27628bb"
-					(reference "R36")
+					(reference "R43")
 					(unit 1)
 				)
@@
 		(in_pos_files yes)
 		(dnp no)
-		(property "Reference" "R50"
+		(property "Reference" "R39"
 			(at 104.14 118.11 0)
 			(show_name no)
@@
 			(project "DronePCB"
 				(path "/c9b74494-ac48-4f27-9459-39f0e04d9d05/064430ba-d2ef-4218-b13a-03feb27628bb"
-					(reference "R50")
+					(reference "R39")
 					(unit 1)
 				)
@@
 		(in_pos_files yes)
 		(dnp no)
-		(property "Reference" "C48"
+		(property "Reference" "C52"
 			(at 146.05 39.7509 0)
 			(show_name no)
@@
 			(project "DronePCB"
 				(path "/c9b74494-ac48-4f27-9459-39f0e04d9d05/064430ba-d2ef-4218-b13a-03feb27628bb"
-					(reference "C48")
+					(reference "C52")
 					(unit 1)
 				)
@@
 		(dnp no)
 		(fields_autoplaced yes)
-		(property "Reference" "R39"
+		(property "Reference" "R46"
 			(at 195.58 69.8499 0)
 			(show_name no)
@@
 			(project "DronePCB"
 				(path "/c9b74494-ac48-4f27-9459-39f0e04d9d05/064430ba-d2ef-4218-b13a-03feb27628bb"
-					(reference "R39")
+					(reference "R46")
 					(unit 1)
 				)
@@
 		(in_pos_files yes)
 		(dnp no)
-		(property "Reference" "R38"
+		(property "Reference" "R45"
 			(at 109.22 142.24 90)
 			(show_name no)
@@
 			(project "DronePCB"
 				(path "/c9b74494-ac48-4f27-9459-39f0e04d9d05/064430ba-d2ef-4218-b13a-03feb27628bb"
-					(reference "R38")
+					(reference "R45")
 					(unit 1)
 				)
@@
 		(dnp no)
 		(fields_autoplaced yes)
-		(property "Reference" "#PWR066"
+		(property "Reference" "#PWR068"
 			(at 180.34 85.09 0)
 			(hide yes)
@@
 			(project "DronePCB"
 				(path "/c9b74494-ac48-4f27-9459-39f0e04d9d05/064430ba-d2ef-4218-b13a-03feb27628bb"
-					(reference "#PWR066")
+					(reference "#PWR068")
 					(unit 1)
 				)
@@
 		(in_pos_files yes)
 		(dnp no)
-		(property "Reference" "C51"
+		(property "Reference" "C55"
 			(at 158.75 118.1099 0)
 			(show_name no)
@@
 			(project "DronePCB"
 				(path "/c9b74494-ac48-4f27-9459-39f0e04d9d05/064430ba-d2ef-4218-b13a-03feb27628bb"
-					(reference "C51")
+					(reference "C55")
 					(unit 1)
 				)
@@
 		(dnp no)
 		(fields_autoplaced yes)
-		(property "Reference" "R40"
+		(property "Reference" "R47"
 			(at 196.85 147.3199 0)
 			(show_name no)
@@
 			(project "DronePCB"
 				(path "/c9b74494-ac48-4f27-9459-39f0e04d9d05/064430ba-d2ef-4218-b13a-03feb27628bb"
-					(reference "R40")
+					(reference "R47")
 					(unit 1)
 				)
@@
 		(in_pos_files yes)
 		(dnp no)
-		(property "Reference" "R45"
+		(property "Reference" "R36"
 			(at 83.82 128.27 90)
 			(show_name no)
@@
 			(project "DronePCB"
 				(path "/c9b74494-ac48-4f27-9459-39f0e04d9d05/064430ba-d2ef-4218-b13a-03feb27628bb"
-					(reference "R45")
+					(reference "R36")
 					(unit 1)
 				)
@@
 		(in_pos_files yes)
 		(dnp no)
-		(property "Reference" "R42"
+		(property "Reference" "R37"
 			(at 87.63 50.8 90)
 			(show_name no)
@@
 			(project "DronePCB"
 				(path "/c9b74494-ac48-4f27-9459-39f0e04d9d05/064430ba-d2ef-4218-b13a-03feb27628bb"
-					(reference "R42")
+					(reference "R37")
 					(unit 1)
 				)
@@
 		(in_pos_files yes)
 		(dnp no)
-		(property "Reference" "C53"
+		(property "Reference" "C57"
 			(at 172.72 118.1099 0)
 			(show_name no)
@@
 			(project "DronePCB"
 				(path "/c9b74494-ac48-4f27-9459-39f0e04d9d05/064430ba-d2ef-4218-b13a-03feb27628bb"
-					(reference "C53")
+					(reference "C57")
 					(unit 1)
 				)
@@
 		(dnp no)
 		(fields_autoplaced yes)
-		(property "Reference" "#PWR065"
+		(property "Reference" "#PWR067"
 			(at 162.56 132.08 0)
 			(hide yes)
@@
 			(project "DronePCB"
 				(path "/c9b74494-ac48-4f27-9459-39f0e04d9d05/064430ba-d2ef-4218-b13a-03feb27628bb"
-					(reference "#PWR065")
+					(reference "#PWR067")
 					(unit 1)
 				)
@@
 		(in_pos_files yes)
 		(dnp yes)
-		(property "Reference" "C47"
+		(property "Reference" "C51"
 			(at 133.35 117.2209 0)
 			(show_name no)
@@
 			(project "DronePCB"
 				(path "/c9b74494-ac48-4f27-9459-39f0e04d9d05/064430ba-d2ef-4218-b13a-03feb27628bb"
-					(reference "C47")
+					(reference "C51")
 					(unit 1)
 				)
@@
 		(in_pos_files yes)
 		(dnp no)
-		(property "Reference" "C50"
+		(property "Reference" "C54"
 			(at 157.48 40.6399 0)
 			(show_name no)
@@
 			(project "DronePCB"
 				(path "/c9b74494-ac48-4f27-9459-39f0e04d9d05/064430ba-d2ef-4218-b13a-03feb27628bb"
-					(reference "C50")
+					(reference "C54")
 					(unit 1)
 				)
@@
 		(in_pos_files yes)
 		(dnp no)
-		(property "Reference" "Q10"
+		(property "Reference" "Q8"
 			(at 119.38 121.9199 0)
 			(show_name no)
@@
 			(project "DronePCB"
 				(path "/c9b74494-ac48-4f27-9459-39f0e04d9d05/064430ba-d2ef-4218-b13a-03feb27628bb"
-					(reference "Q10")
+					(reference "Q8")
 					(unit 1)
 				)
@@
 		(in_pos_files yes)
 		(dnp no)
-		(property "Reference" "C49"
+		(property "Reference" "C53"
 			(at 147.32 117.2209 0)
 			(show_name no)
@@
 			(project "DronePCB"
 				(path "/c9b74494-ac48-4f27-9459-39f0e04d9d05/064430ba-d2ef-4218-b13a-03feb27628bb"
-					(reference "C49")
+					(reference "C53")
 					(unit 1)
 				)
@@
 		(in_pos_files yes)
 		(dnp no)
-		(property "Reference" "C52"
+		(property "Reference" "C56"
 			(at 171.45 40.6399 0)
 			(show_name no)
@@
 			(project "DronePCB"
 				(path "/c9b74494-ac48-4f27-9459-39f0e04d9d05/064430ba-d2ef-4218-b13a-03feb27628bb"
-					(reference "C52")
+					(reference "C56")
 					(unit 1)
 				)
@@
 		(in_pos_files yes)
 		(dnp no)
-		(property "Reference" "Q9"
+		(property "Reference" "Q7"
 			(at 119.38 69.8501 0)
 			(show_name no)
@@
 			(project "DronePCB"
 				(path "/c9b74494-ac48-4f27-9459-39f0e04d9d05/064430ba-d2ef-4218-b13a-03feb27628bb"
-					(reference "Q9")
+					(reference "Q7")
 					(unit 1)
 				)
@@
 		(in_pos_files yes)
 		(dnp no)
-		(property "Reference" "R44"
+		(property "Reference" "R38"
 			(at 109.22 77.47 0)
 			(show_name no)
@@
 			(project "DronePCB"
 				(path "/c9b74494-ac48-4f27-9459-39f0e04d9d05/064430ba-d2ef-4218-b13a-03feb27628bb"
-					(reference "R44")
+					(reference "R38")
 					(unit 1)
 				)
@@
 		(dnp no)
 		(fields_autoplaced yes)
-		(property "Reference" "#PWR064"
+		(property "Reference" "#PWR066"
 			(at 161.29 54.61 0)
 			(hide yes)
@@
 			(project "DronePCB"
 				(path "/c9b74494-ac48-4f27-9459-39f0e04d9d05/064430ba-d2ef-4218-b13a-03feb27628bb"
-					(reference "#PWR064")
+					(reference "#PWR066")
 					(unit 1)
 				)
@@
 		(in_pos_files yes)
 		(dnp no)
-		(property "Reference" "R46"
+		(property "Reference" "R40"
 			(at 109.22 154.94 0)
 			(show_name no)
@@
 			(project "DronePCB"
 				(path "/c9b74494-ac48-4f27-9459-39f0e04d9d05/064430ba-d2ef-4218-b13a-03feb27628bb"
-					(reference "R46")
+					(reference "R40")
 					(unit 1)
 				)
@@
 		(in_pos_files yes)
 		(dnp no)
-		(property "Reference" "Q11"
+		(property "Reference" "Q9"
 			(at 119.38 147.3201 0)
 			(show_name no)
@@
 			(project "DronePCB"
 				(path "/c9b74494-ac48-4f27-9459-39f0e04d9d05/064430ba-d2ef-4218-b13a-03feb27628bb"
-					(reference "Q11")
-					(unit 1)
-				)
+					(reference "Q9")
+					(unit 1)
+				)
