File: DronePCB/DronePCB.kicad_pcb (KiCad board)
At the start: 4 copper layers, 158 x 68 mm, 157 parts, among them J1 VBUS, J10 SysPower, J2 PD_SCL, J3 PD_SDA, J4 SysPower, J5 UART, J6 5V, J7 3V3, J8 USB_C_Receptacle_PowerOnly_6P, J9 Batt, M1 Motor_DC, M2 Motor_DC, Q1 AO3400A, Q2 AO3400A, Q3 AO3400A, Q4 AO3400A, Q5 AO3400A, Q6 AO3401A, Q7 AO3401A, Q8 AO3401A, Q9 AO3401A, U1 RASPBERRY_PI_ZERO_2_W, U10 DRV8231DDAR, U2 CC1101RGPR, U3 BQ24725A, U4 CYPD3177-24LQXQT, U5 DMP3098LSD-13, U6 DMP3098LSD-13, U7 LMR33630BDDA, U8 TSOP45xx, U9 DRV8231DDAR, Y1 NX3225GA

Commit message: Added finishing details to PCB
Parts:
- added G***: LOGO, LOGO, F.Cu at (102.0, 61.0)
- added GND: TestPoint_Pad_D2.0mm, TestPoint:TestPoint_Pad_D2.0mm, F.Cu at (109.0, 96.0)
- added REF**: MountingHole_2.2mm_M2_DIN965_Pad_TopBottom, MountingHole:MountingHole_2.2mm_M2_DIN965_Pad_TopBottom, F.Cu at (97.0, 112.0)
- added REF**: MountingHole_2.2mm_M2_DIN965_Pad_TopBottom, MountingHole:MountingHole_2.2mm_M2_DIN965_Pad_TopBottom, F.Cu at (247.0, 112.0)
- added REF**: MountingHole_2.2mm_M2_DIN965_Pad_TopBottom, MountingHole:MountingHole_2.2mm_M2_DIN965_Pad_TopBottom, F.Cu at (97.0, 52.0)
- added VDD: TestPoint_Pad_D2.0mm, TestPoint:TestPoint_Pad_D2.0mm, F.Cu at (116.0, 96.0)
Routing:
- net VDD: track 1.67 -> 7.67 mm, vias 30 -> 33
Other:
- outline, holes or cut-outs redrawn
- board text added: "DRONE OUT!"
- board text added: "EE300W Spring 2026"
- board text added: "{dblquote}It's drone phase not phone phase{dblquote}"

Commit message: Finalized Drone PCB
Parts:
- added 5V: TestPoint_Pad_D2.0mm, TestPoint:TestPoint_Pad_D2.0mm, F.Cu at (151.5, 75.5)
- added GND: TestPoint_Pad_D2.0mm, TestPoint:TestPoint_Pad_D2.0mm, F.Cu at (109.0, 101.0)
- added GND: TestPoint_Pad_D2.0mm, TestPoint:TestPoint_Pad_D2.0mm, F.Cu at (109.0, 106.0)
- added SP: TestPoint_Pad_D2.0mm, TestPoint:TestPoint_Pad_D2.0mm, F.Cu at (150.5, 111.5)
- moved G*** 3.16 mm to (101.0, 58.0)
- renumbered AE1 to 315MHz
Routing:
- net /CC1101Radio/MOSI: track 50.4 -> 51.3 mm
- net /I2S Microphone/WS: track 65.0 -> 64.3 mm
- net Net-(D1-K): track 14.9 -> 15.0 mm, vias 0 -> 2
Other:
- board text added: "3s2p Li-Ion Battery Charger"
- board text added: "Brenden"
- board text added: "CC1101 Sub-GHz Radio"
- board text added: "H-Bridge Motor Driver (L)"
- board text added: "H-Bridge Motor Driver (R)"
- board text added: "I2S Mic"
- board text added: "IR Remote Emulator + Blaster"
- board text added: "Ioannis"
- board text added: "Matt"
- board text added: "Nick"
- board text added: "Rev. 0"
- board text added: "Test Pads"
- board text added: "USB-C PD"
