File: DronePCB/BatteryCharger/Battery_Charger.kicad_sch (KiCad schematic)
At the start: 43 parts, among them Q1 AO3400A, Q2 AO3400A, Q5 AO3400A, U1 BQ24725A

Commit message: All circuits complete
Parts:
- removed Ci: 2.2 uF, symbol Device:C
- removed Csys: 220 uF, symbol Device:C
- removed R3, R4: 10 k ohms, symbol Device:R
- removed Ri: 2 ohms, symbol Device:R
- added J9: Batt, Connector_Wire:SolderWire-0.25sqmm_1x02_P4.2mm_D0.65mm_OD1.7mm_Relief, symbol Connector:Conn_01x02_Socket
- C18: renamed from C17; footprint (none) -> Capacitor_SMD:C_1210_3225Metric
- C19: renamed from C16; footprint (none) -> Capacitor_SMD:C_0603_1608Metric
- C20: renamed from C1; footprint (none) -> Capacitor_SMD:C_0603_1608Metric
- C21: renamed from C2; footprint (none) -> Capacitor_SMD:C_0603_1608Metric
- C22: renamed from C3; footprint (none) -> Capacitor_SMD:C_0603_1608Metric
- C23: renamed from C4; footprint (none) -> Capacitor_SMD:C_0603_1608Metric
- C24: renamed from C7; footprint (none) -> Capacitor_SMD:C_0603_1608Metric
- C25: renamed from C6; footprint (none) -> Capacitor_SMD:C_0603_1608Metric
- C26: renamed from C5; footprint (none) -> Capacitor_SMD:C_0603_1608Metric
- C27: renamed from C13; footprint (none) -> Capacitor_SMD:C_0603_1608Metric
- C28: renamed from C14; footprint (none) -> Capacitor_SMD:C_0603_1608Metric
- C29: renamed from C8; footprint (none) -> Capacitor_SMD:C_1206_3216Metric
- C30: renamed from C9; footprint (none) -> Capacitor_SMD:C_1206_3216Metric
- C31: renamed from C15; footprint (none) -> Capacitor_SMD:C_0603_1608Metric
- C32: renamed from C10; footprint (none) -> Capacitor_SMD:C_1206_3216Metric
- C33: renamed from C11; footprint (none) -> Capacitor_SMD:C_1206_3216Metric
- L5: renamed from L1; footprint (none) -> Inductor_SMD:L_Vishay_IHLP-2525
- MOSFET1: renamed from MOSFET2; footprint POWERPAK_1212-8 -> Package_SO:Vishay_PowerPAK_1212-8_Single
- MOSFET2: renamed from MOSFET1; footprint POWERPAK_1212-8 -> Package_SO:Vishay_PowerPAK_1212-8_Single
- Q1, Q2: footprint FDS6680A:SOIC127P600X175-8N -> Package_SO:SO-8_3.9x4.9mm_P1.27mm
- Q3: renamed from Q5; footprint FDS6680A:SOIC127P600X175-8N -> Package_SO:SO-8_3.9x4.9mm_P1.27mm
- R11: renamed from R8; footprint (none) -> Resistor_SMD:R_0603_1608Metric
- R12: renamed from R7; footprint (none) -> Resistor_SMD:R_0603_1608Metric
- R13: renamed from R5; footprint (none) -> Resistor_SMD:R_0603_1608Metric
- R14: renamed from R9; footprint (none) -> Resistor_SMD:R_0603_1608Metric
- R15: renamed from R6; footprint (none) -> Resistor_SMD:R_0603_1608Metric
- R16: renamed from R14; footprint (none) -> Resistor_SMD:R_0603_1608Metric
- R17: renamed from R15; footprint (none) -> Resistor_SMD:R_0603_1608Metric
- R5: renamed from R1; footprint (none) -> Resistor_SMD:R_0603_1608Metric
- R6: renamed from R2; footprint (none) -> Resistor_SMD:R_0603_1608Metric
- R7: renamed from R10; footprint (none) -> Resistor_SMD:R_0603_1608Metric
- R9: renamed from R11; footprint (none) -> Resistor_SMD:R_0603_1608Metric
- RAC1: renamed from RAC; footprint (none) -> Resistor_SMD:R_0603_1608Metric
- RSR1: renamed from RSR; footprint (none) -> Resistor_SMD:R_0603_1608Metric
- U3: renamed from U1; footprint (none) -> ExternalParts:QFN50P350X350X100-21N
Connections:
- net VBUS: now reaches C18.1, D2.1, Q1.5, Q1.6, Q1.7, Q1.8, R5.1
- net SystemPower: now reaches C21.1, C22.1, C29.1, C30.1, D2.2, MOSFET2.8 (D), Q3.5, Q3.6, Q3.7, Q3.8, RAC1.2, U3.1 (ACN)
- net SystemPower: now also MOSFET2.5 (D), MOSFET2.6 (D), MOSFET2.7 (D)
- net at C24.2, L5.1, MOSFET1.8 (D)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: now also MOSFET1.5 (D), MOSFET1.6 (D), MOSFET1.7 (D), MOSFET2.2 (S), MOSFET2.3 (S)
- net ACOK: now reaches R13.2, U3.5 (ACOK)
- net SDA: now reaches U3.8 (SDA)
- net SCL: now reaches U3.9 (SCL)
- net at C32.1, C33.1, RSR1.2: now also C27.2, C28.1, C31.2, Q3.1, Q3.2, Q3.3, R17.1, J9.1 (Pin_1)
- net GND: now reaches MOSFET1.2 (S)
- net GND: now also C20.2, C22.2, C23.2, C25.1, C26.2, C28.2, C29.2, C30.2, C32.2, C33.2, MOSFET1.1 (S), MOSFET1.3 (S), R11.2, R6.2, U3.14 (GND), U3.21 (PowerPad), J9.2 (Pin_2)
- net +3.3V renamed +3.3
- removed net GND1: C20.2, C22.2, C23.2, C25.1, C26.2, C28.2, C29.2, C30.2, C32.2, C33.2, MOSFET1.1 (S), R11.2, R6.2, U3. (PowerPad), U3.14 (GND)
Other:
- note removed: "Adapter +"
- moved on the sheet: C22
